File: EagleFiles/SDDD-PulseBoard-1.0.sch (EAGLE design)
At the start: 39 parts, among them IC1 NE555, IC2 NE555, IC3 IR4426, IC4 7812TV, IC5 IR4426, Q1 IRFB3307, Q2 IRFB3307, Q3 IRFB3307, T1 2N2907

Commit message: Add files via upload
Parts:
- C6, C7, C8, C9: value 0.1µf -> 0.01µf
Changed lines of the file:
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@@
 <part name="R4" library="resistor" deviceset="R-EU_" device="0207/10" value="10k"/>
 <part name="R5" library="resistor" deviceset="R-EU_" device="0207/10" value="100"/>
-<part name="C6" library="rcl" deviceset="C-EU" device="050-025X075" value="0.1µf"/>
-<part name="C7" library="rcl" deviceset="C-EU" device="050-025X075" value="0.1µf"/>
-<part name="C8" library="rcl" deviceset="C-EU" device="050-025X075" value="0.1µf"/>
+<part name="C6" library="rcl" deviceset="C-EU" device="050-025X075" value="0.01µf"/>
+<part name="C7" library="rcl" deviceset="C-EU" device="050-025X075" value="0.01µf"/>
+<part name="C8" library="rcl" deviceset="C-EU" device="050-025X075" value="0.01µf"/>
 <part name="R6" library="resistor" deviceset="R-EU_" device="0207/10" value="3k"/>
-<part name="C9" library="rcl" deviceset="C-EU" device="050-025X075" value="0.1µf"/>
+<part name="C9" library="rcl" deviceset="C-EU" device="050-025X075" value="0.01µf"/>
 <part name="IC1" library="st-microelectronics" deviceset="NE555" device=""/>
 <part name="IC2" library="st-microelectronics" deviceset="NE555" device=""/>
